File: design_files/AST1030.brd (EAGLE design)
At the start: 10 x 10 mm, 6 parts, among them J1 SM05B, M1 SPW2430

Commit message: name change
Parts:
- C1: value 0.1uF -> 1uF; device tinycircuits:C0402 -> tinycircuits:C0603
- C2: value 10uF -> 0.1uF; device tinycircuits:C0603 -> tinycircuits:C0402
- J1: device tinycircuits:JST_SH_5X1 -> tinycircuits:JST_SH_5X1_EDGE
- moved C1 2.29 mm to (16.9, 16.2), turned to 180 degrees
- moved C2 2.29 mm to (18.2, 18.1), turned to 90 degrees
- renumbered M1 to U1
Other:
- board text added: "Wireling Microphone"
- board text removed: "Microphone Board"
Changed lines of the file:
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@@
 <layer number="59" name="Invisible" color="7" fill="1" visible="no" active="no"/>
 <layer number="61" name="stand" color="7" fill="1" visible="no" active="no"/>
+<layer number="88" name="SimResults" color="9" fill="1" visible="yes" active="yes"/>
+<layer number="89" name="SimProbes" color="9" fill="1" visible="yes" active="yes"/>
 <layer number="90" name="Modules" color="5" fill="1" visible="yes" active="yes"/>
 <layer number="91" name="Nets" color="2" fill="1" visible="no" active="no"/>
@@
 <layer number="158" name="bResistor" color="7" fill="1" visible="no" active="yes"/>
 <layer number="159" name="henwayCAP" color="13" fill="1" visible="yes" active="yes"/>
+<layer number="160" name="IDFDebug" color="7" fill="1" visible="yes" active="yes"/>
 <layer number="191" name="mNets" color="7" fill="1" visible="no" active="no"/>
 <layer number="192" name="mBusses" color="7" fill="1" visible="no" active="no"/>
@@
 <wire x1="0" y1="40.8" x2="0" y2="0" width="0.127" layer="48"/>
 <dimension x1="15" y1="20" x2="25" y2="20" x3="20" y3="21.454653125" layer="48"/>
-<text x="38.111025" y="4.365003125" size="0.889" layer="48">Microphone Board</text>
+<text x="38.111025" y="4.365003125" size="0.889" layer="48">Wireling Microphone</text>
 <text x="34.986825" y="1.7714" size="0.889" layer="48">AS-PCB-AST1030</text>
 <text x="57.3810375" y="1.6952" size="0.889" layer="48">1</text>
@@
 <attribute name="NO_BOM" value="TRUE" x="34" y="0" size="1.778" layer="27" display="off"/>
 </element>
-<element name="C1" library="tinycircuits" package="C0402" value="0.1uF" x="18.25" y="18.05" rot="R90">
+<element name="C2" library="tinycircuits" package="C0402" value="0.1uF" x="18.25" y="18.05" rot="R90">
 <attribute name="PARTNO" value="AS-ITM-00008" x="18.25" y="18.05" size="1.778" layer="27" rot="R90" display="off"/>
 <attribute name="VALUE" value="0.1uF" x="18.25" y="18.05" size="1.778" layer="27" rot="R90" display="off"/>
 </element>
-<element name="C2" library="tinycircuits" package="C0603" value="10uF" x="16.9" y="16.2" rot="R180">
-<attribute name="PARTNO" value="AS-ITM-00002" x="16.9" y="16.2" size="1.778" layer="27" rot="R180" display="off"/>
-<attribute name="VALUE" value="10uF" x="16.9" y="16.2" size="1.778" layer="27" rot="R180" display="off"/>
+<element name="C1" library="tinycircuits" package="C0603" value="1uF" x="16.9" y="16.2" rot="R180">
+<attribute name="PARTNO" value="AS-ITM-00410" x="16.9" y="16.2" size="1.778" layer="27" rot="R180" display="off"/>
+<attribute name="VALUE" value="1uF" x="16.9" y="16.2" size="1.778" layer="27" rot="R180" display="off"/>
 </element>
-<element name="J1" library="tinycircuits" package="JST_SH_5X1" value="SM05B" x="20" y="12.125">
+<element name="J1" library="tinycircuits" package="JST_SH_5X1_EDGE" value="SM05B" x="20" y="12.125">
 <attribute name="PARTNO" value="AS-ITM-00340" x="20" y="12.125" size="1.778" layer="27" display="off"/>
 <attribute name="VALUE" value="SM05B" x="20" y="12.125" size="1.778" layer="27" display="off"/>
@@
 <attribute name="VALUE" value="1.00K" x="23.5" y="15.9" size="1.778" layer="27" rot="R270" display="off"/>
 </element>
-<element name="M1" library="tinycircuits" package="SPW2430HR5H-B" value="SPW2430" x="20.2" y="17.7" rot="R180">
+<element name="U1" library="tinycircuits" package="SPW2430HR5H-B" value="SPW2430" x="20.2" y="17.7" rot="R180">
 <attribute name="PARTNO" value="AS-ITM-00387" x="20.2" y="17.7" size="1.778" layer="27" rot="R180" display="off"/>
 <attribute name="VALUE" value="SPW2430" x="20.2" y="17.7" size="1.778" layer="27" rot="R180" display="off"/>
@@
 <vertex x="15" y="10"/>
 </polygon>
-<contactref element="C1" pad="2"/>
 <contactref element="C2" pad="2"/>
+<contactref element="C1" pad="2"/>
 <contactref element="J1" pad="1"/>
 <via x="18.1" y="10.7" extent="1-16" drill="0.381"/>
 <via x="21.9" y="10.6" extent="1-16" drill="0.381"/>
-<contactref element="M1" pad="3"/>
-<contactref element="M1" pad="2"/>
-<via x="17" y="14.1" extent="1-16" drill="0.381"/>
+<contactref element="U1" pad="3"/>
+<contactref element="U1" pad="2"/>
+<via x="16.1" y="14.5" extent="1-16" drill="0.381"/>
 <via x="22.1" y="18.1" extent="1-16" drill="0.381"/>
 <via x="17.1" y="17.3" extent="1-16" drill="0.381"/>
@@
 </signal>
 <signal name="VCC">
-<contactref element="C1" pad="1"/>
 <contactref element="C2" pad="1"/>
+<contactref element="C1" pad="1"/>
 <contactref element="J1" pad="2"/>
-<contactref element="M1" pad="4"/>
+<contactref element="U1" pad="4"/>
 <wire x1="19.5" y1="16.51" x2="19.525" y2="16.485" width="0.3048" layer="1"/>
 <wire x1="18.25" y1="17.4" x2="19.51" y2="16.5" width="0.3048" layer="1"/>
@@
 <signal name="N$2">
 <contactref element="R1" pad="1"/>
-<contactref element="M1" pad="1"/>
+<contactref element="U1" pad="1"/>
 <wire x1="20.875" y1="16.485" x2="23.485" y2="16.485" width="0.3048" layer="1"/>
 <wire x1="23.485" y1="16.485" x2="23.5" y2="16.5" width="0.3048" layer="1"/>
