File: design_files/AST1030.sch (EAGLE design)
At the start: 5 parts, among them J1 SM05B, M1 SPW2430

Commit message: name change
Parts:
- C1: value 0.1uF -> 1uF; device tinycircuits:AS-ITM-00008 -> tinycircuits:AS-ITM-00410; PARTNO (none) -> AS-ITM-00410; VALUE (none) -> 1uF
- C2: value 10uF -> 0.1uF; device tinycircuits:AS-ITM-00002 -> tinycircuits:AS-ITM-00008
- J1: device tinycircuits:AS-ITM-00340 -> tinycircuits:AS-ITM-00340EDGE
- renumbered M1 to U1
Other:
- note added: "Wireling Microphone"
- note removed: "Microphone Board"
- moved on the sheet: C1, C2

Commit message: updated documentation
Other:
- note added: "Variant: Standard - R"
- note removed: "Variant: Standard"
Changed lines of the file:
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@@
 <text x="63.5" y="66.04" size="1.778" layer="96">Hand Populated: -</text>
 <text x="63.5" y="63.5" size="1.778" layer="96">Hand Soldered: -</text>
-<text x="63.5" y="71.12" size="1.778" layer="96">Variant: Standard</text>
+<text x="63.5" y="71.12" size="1.778" layer="96">Variant: Standard - R</text>
 <text x="63.5" y="60.96" size="1.778" layer="96">Notes: -</text>
 </plain>
